File: ReflowToasterOven2.kicad_pcb (KiCad board)
At the start: 4 copper layers, 114.3 x 45.8 mm, 15 parts, among them P1 Buzzer, P2 Switches, T1 Thermocouple, T2 5V Power, T3 Relay, U1 FEATHER_M0_EXPRESS, U2 AD595AQ

Commit message: Label Update
Parts:
- T1: value Thermocouple -> + Therm -
Changed lines of the file:
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@@
     (links 33)
     (no_connects 0)
-    (area 55.829999 91.349999 170.230001 137.210001)
+    (area 26.785994 89.31148 199.472126 139.38758)
     (thickness 1.6)
     (drawings 4)
@@
       (effects (font (size 1.524 1.524) (thickness 0.3048)))
     )
-    (fp_text value Thermocouple (at 0 5.842) (layer F.SilkS)
+    (fp_text value "+ Therm -" (at 0 5.842) (layer F.SilkS)
       (effects (font (size 1.524 1.524) (thickness 0.3048)))
     )
