File: ReflowToasterOven2.sch (KiCad schematic (older format))
At the start: 11 parts, among them P1 Buzzer, P2 Switches, T1 Thermocouple, T2 5V Power, T3 Relay, U1 FEATHER_M0_EXPRESS, U2 AD595AQ

Commit message: Label Update
Parts:
- T1: value Thermocouple -> + Therm -
Changed lines of the file:
@@
 Sheet 1 1
 Title ""
-Date "24 jun 2018"
+Date "26 jun 2018"
 Rev ""
 Comp ""
@@
 P 1050 4300
 F 0 "T1" V 1000 4300 40  0000 C CNN
-F 1 "Thermocouple" V 1100 4300 40  0000 C CNN
+F 1 "+ Therm -" V 1100 4300 40  0000 C CNN
 F 2 "~" H 1050 4300 60  0000 C CNN
 F 3 "~" H 1050 4300 60  0000 C CNN
